Commit message: LIDAR added and working!

File: description/robot.urdf.xacro (robot description, xacro)
@@ -3,3 +3,4 @@
    <xacro:include filename="robot_core.xacro"/>
    <xacro:include filename="gazebo_control.xacro"/>
+   <xacro:include filename="lidar.xacro"/>
 </robot>

File: description/robot_core.xacro (robot description, xacro)
@@ -13,4 +13,7 @@
     <material name="black">
     <color rgba="0 0 0 1"/>
+    </material>
+    <material name="red">
+    <color rgba="1 0 0 1"/>
     </material>
     <!-- Center of the two drive wheels/centr of rotation-->

Commit message: ros2 control updates and fixes

File: description/robot.urdf.xacro (robot description, xacro)
@@ -1,9 +1,14 @@
 <?xml version="1.0"?>
 <robot xmlns:xacro="http://www.ros.org/wiki/xacro"  name="robot">
+   <xacro:arg name="use_ros2_control" default="true"/>
    <xacro:include filename="robot_core.xacro"/>
-   <!-- <xacro:include filename="gazebo_control.xacro"/> -->
-   <xacro:include filename="ros2_control.xacro"/>
-   <xacro:include filename="lidar.xacro"/>
-   <!-- <xacro:include filename="camera.xacro"/> -->
-   <xacro:include filename="depth_camera.xacro"/>
+   <xacro:if value="$(arg use_ros2_control)">
+        <xacro:include filename="ros2_control.xacro" />
+   </xacro:if>
+    <xacro:unless value="$(arg use_ros2_control)">
+        <xacro:include filename="gazebo_control.xacro" />
+    </xacro:unless>
+    <xacro:include filename="lidar.xacro" />
+    <xacro:include filename="camera.xacro" />
+   <!-- <xacro:include filename="depth_camera.xacro"/> -->
 </robot>

File: description/robot_core.xacro (robot description, xacro)
@@ -64,5 +64,5 @@
         <collision>
             <geometry>
-                <cylinder radius="0.05" length="0.04"/>
+                <sphere radius="0.05"/>
             </geometry>
         </collision>
@@ -90,5 +90,5 @@
         <collision>
             <geometry>
-                <cylinder radius="0.05" length="0.04"/>
+                <sphere radius="0.05"/>
             </geometry>
         </collision>

Commit message: gazebo updates for sim time

File: description/robot.urdf.xacro (robot description, xacro)
@@ -2,4 +2,5 @@
 <robot xmlns:xacro="http://www.ros.org/wiki/xacro"  name="robot">
    <xacro:arg name="use_ros2_control" default="true"/>
+   <xacro:arg name="sim_mode" default="false"/>
    <xacro:include filename="robot_core.xacro"/>
    <xacro:if value="$(arg use_ros2_control)">

File: description/ros2_control.xacro (robot description, xacro)
@@ -1,56 +1,61 @@
 <?xml version="1.0"?>
 <robot xmlns:xacro="http://www.ros.org/wiki/xacro"  name="robot">
-<ros2_control name="RealRobot" type="system">
-    <hardware>
-        <plugin>diffdrive_arduino/DiffDriveArduino</plugin>
-        <param name="left_wheel_name">left_wheel_joint</param>
-        <param name="right_wheel_name">right_wheel_joint</param>
-        <param name="loop_rate">30</param>
-        <param name="device">/dev/ttyUSB0</param>
-        <param name="baud_rate">57600</param>
-        <param name="timeout">1000</param>
-        <param name="enc_counts_per_rev">3436</param>
-    </hardware>
-    <joint name="left_wheel_joint">
-        <command_interface name="velocity">
-            <param name="min">-10</param>
-            <param name="max">10</param>
-        </command_interface>
-            <state_interface name="velocity"/>
-            <state_interface name="position"/>
-    </joint>
-    <joint name="right_wheel_joint">
-        <command_interface name="velocity">
-            <param name="min">-10</param>
-            <param name="max">10</param>
-        </command_interface>
-            <state_interface name="velocity"/>
-            <state_interface name="position"/>
-    </joint>
-</ros2_control>
-<!-- <ros2_control name="GazeboSystem" type="system">
-    <hardware>
-        <plugin>gazebo_ros2_control/GazeboSystem</plugin>
-    </hardware>
-    <joint name="left_wheel_joint">
-        <command_interface name="velocity">
-            <param name="min">-10</param>
-            <param name="max">10</param>
-        </command_interface>
-            <state_interface name="velocity"/>
-            <state_interface name="position"/>
-    </joint>
-    <joint name="right_wheel_joint">
-        <command_interface name="velocity">
-            <param name="min">-10</param>
-            <param name="max">10</param>
-        </command_interface>
-            <state_interface name="velocity"/>
-            <state_interface name="position"/>
-    </joint>
-</ros2_control> -->
+<xacro:unless value="$(arg sim_mode)">
+    <ros2_control name="RealRobot" type="system">
+        <hardware>
+            <plugin>diffdrive_arduino/DiffDriveArduino</plugin>
+            <param name="left_wheel_name">left_wheel_joint</param>
+            <param name="right_wheel_name">right_wheel_joint</param>
+            <param name="loop_rate">30</param>
+            <param name="device">/dev/ttyUSB0</param>
+            <param name="baud_rate">57600</param>
+            <param name="timeout">1000</param>
+            <param name="enc_counts_per_rev">3436</param>
+        </hardware>
+        <joint name="left_wheel_joint">
+            <command_interface name="velocity">
+                <param name="min">-10</param>
+                <param name="max">10</param>
+            </command_interface>
+                <state_interface name="velocity"/>
+                <state_interface name="position"/>
+        </joint>
+        <joint name="right_wheel_joint">
+            <command_interface name="velocity">
+                <param name="min">-10</param<xacro:if value="$(arg use_ros2_control)">
+                <param name="max">10</param>
+            </command_interface>
+                <state_interface name="velocity"/>
+                <state_interface name="position"/>
+        </joint>
+    </ros2_control>
+</xacro:unless>>
+<xacro:if value="$(arg sim_mode)">
+    <ros2_control name="GazeboSystem" type="system">
+        <hardware>
+            <plugin>gazebo_ros2_control/GazeboSystem</plugin>
+        </hardware>
+        <joint name="left_wheel_joint">
+            <command_interface name="velocity">
+                <param name="min">-10</param>
+                <param name="max">10</param>
+            </command_interface>
+                <state_interface name="velocity"/>
+                <state_interface name="position"/>
+        </joint>
+        <joint name="right_wheel_joint">
+            <command_interface name="velocity">
+                <param name="min">-10</param>
+                <param name="max">10</param>
+            </command_interface>
+                <state_interface name="velocity"/>
+                <state_interface name="position"/>
+        </joint>
+    </ros2_control>
+</xacro:if>
     <gazebo>
         <plugin name="gazebo_ros2_control" filename="libgazebo_ros2_control.so">
             <parameters>$(find articubot_one)/config/my_controllers.yaml</parameters>
+            <parameters>$(find articubot_one)/config/gaz_ros2_ctl_use_sim.yaml</parameters>
         </plugin>
     </gazebo>
