Commit message: Fixed steering and Lidar position on bot

File: description/lidar.xacro (robot description, xacro)
@@ -4,5 +4,5 @@
     <parent link="chassis"/>
     <child link="laser_frame"/>
-    <origin xyz="0.1 0 0.175" rpy="0 0 0"/>
+    <origin xyz="0.18 0 0.1485" rpy="0 0 0"/>
 </joint>
 <link name="laser_frame">

File: description/robot_core.xacro (robot description, xacro)
@@ -31,5 +31,5 @@
         <color rgba="1 0 0 1"/>
     </material>
-    <!-- Center of the two drive wheels/centr of rotation-->
+    <!-- Center of the two drive wheels/center of rotation-->
     <link name="base_link">
     </link>
@@ -74,6 +74,6 @@
         <parent link="base_link"/>
         <child link="left_wheel"/>
-        <origin xyz="0 ${-wheel_offset_y} 0" rpy="-${pi/2} 0 0" />
-        <axis xyz="0 0 1"/>
+        <origin xyz="0 ${wheel_offset_y} 0" rpy="${pi/2} 0 0" />
+        <axis xyz="0 0 -1"/>
     </joint>
     <link name="left_wheel">
@@ -100,6 +100,6 @@
         <parent link="base_link"/>
         <child link="right_wheel"/>
-        <origin xyz="0 ${wheel_offset_y} 0" rpy="${pi/2} 0 0" />
-        <axis xyz="0 0 -1"/>
+        <origin xyz="0 ${-wheel_offset_y} 0" rpy="-${pi/2} 0 0" />
+        <axis xyz="0 0 1"/>
     </joint>
     <link name="right_wheel">

File: description/ros2_control.xacro (robot description, xacro)
@@ -15,6 +15,6 @@
         <joint name="left_wheel_joint">
             <command_interface name="velocity">
-                <param name="min">-10</param>
-                <param name="max">10</param>
+                <param name="min">10</param>
+                <param name="max">-10</param>
             </command_interface>
                 <state_interface name="velocity"/>
@@ -23,6 +23,6 @@
         <joint name="right_wheel_joint">
             <command_interface name="velocity">
-                <param name="min">-10</param>
-                <param name="max">10</param>
+                <param name="min">10</param>
+                <param name="max">-10</param>
             </command_interface>
                 <state_interface name="velocity"/>
@@ -38,6 +38,6 @@
         <joint name="left_wheel_joint">
             <command_interface name="velocity">
-                <param name="min">-10</param>
-                <param name="max">10</param>
+                <param name="min">10</param>
+                <param name="max">-10</param>
             </command_interface>
                 <state_interface name="velocity"/>
@@ -46,6 +46,6 @@
         <joint name="right_wheel_joint">
             <command_interface name="velocity">
-                <param name="min">-10</param>
-                <param name="max">10</param>
+                <param name="min">10</param>
+                <param name="max">-10</param>
             </command_interface>
                 <state_interface name="velocity"/>
