Commit message: camera working

File: description/camera.xacro (robot description, xacro)
@@ -4,5 +4,5 @@
     <parent link="chassis"/>
     <child link="camera_link"/>
-    <origin xyz="0.305 0 0.8" rpy="0 0 0"/>
+    <origin xyz="0.305 0 0.08" rpy="0 0 0"/>
 </joint>
 <link name="camera_link">
@@ -19,34 +19,27 @@
     <origin xyz="0 0 0" rpy="${-pi/2} 0 ${-pi/2}"/>
 </joint>
-<link name="camera_link"></link>
+<link name="camera_link_optical"></link>
     <gazebo reference="camera_link">
         <material>Gazebo/Red</material>
-        <!-- <sensor name="laser" type="ray">
+        <sensor name="camera" type="camera">
         <pose> 0 0 0 0 0 0 </pose>
         <visualize>true</visualize>
         <update_rate>10</update_rate>
-        <ray>
-            <scan>
-                <horizontal>
-                    <samples>360</samples>
-                    <resolution>1</resolution>
-                    <min_angle>-3.14</min_angle>
-                    <max_angle>3.14</max_angle>
-                </horizontal>
-            </scan>
-            <range>
-                <min>0.3</min>
-                <max>12</max>
-                <resolution>0.01</resolution>
-            </range>
-        </ray>
-        <plugin name="laser_controller" filename="libgazebo_ros_ray_sensor.so">
-            <ros>
-                <argument>~/out:=scan</argument>
-            </ros>
-            <output_type>sensor_msgs/LaserScan</output_type>
-            <frame_name>laser_frame</frame_name>
+        <camera>
+            <horizontal_fov>1.089</horizontal_fov>
+            <image>
+                <format>R8G8B8</format>
+                <width>640</width>
+                <height>480</height>
+            </image>
+            <clip>
+                <near>0.05</near>
+                <far>8.0</far>
+            </clip>
+        </camera>
+        <plugin name="camera_controller" filename="libgazebo_ros_camera.so">
+            <frame_name>camera_link_optical</frame_name>
         </plugin>
-        </sensor> -->
+        </sensor>
         </gazebo>
 </robot>

File: description/lidar.xacro (robot description, xacro)
@@ -26,5 +26,5 @@
         <sensor name="laser" type="ray">
         <pose> 0 0 0 0 0 0 </pose>
-        <visualize>true</visualize>
+        <visualize>false</visualize>
         <update_rate>10</update_rate>
         <ray>

Commit message: add ball tracker and launch files

File: description/camera.xacro (robot description, xacro)
@@ -4,5 +4,5 @@
     <parent link="chassis"/>
     <child link="camera_link"/>
-    <origin xyz="0.305 0 0.08" rpy="0 0 0"/>
+    <origin xyz="0.305 0 0.08" rpy="0 0.18 0"/>
 </joint>
 <link name="camera_link">
